Commit message: Remove kuka_kr210_k_ultra_support package and add config to kuka_kr210_support instead.

File: kuka_kr210_support/urdf/kr210r3300kultra.urdf (robot description, URDF)
Before this commit: robot kr210_r3300_k_ultra, 7 links, 6 joints
Links:
- removed link a1
- removed link a2
- removed link a3
- removed link a4
- removed link a5
- removed link a6
- added link link_a1, mass 146.16; collision mesh filename=package://kuka_kr210_support/meshes/kr210r3300kultra/link_a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; visual mesh filename=package://kuka_kr210_support/meshes/kr210r3300kultra/link_a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
- added link link_a2, mass 126.48; collision mesh filename=package://kuka_kr210_support/meshes/kr210r3300kultra/link_a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; visual mesh filename=package://kuka_kr210_support/meshes/kr210r3300kultra/link_a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
- added link link_a3, mass 85.793; collision mesh filename=package://kuka_kr210_support/meshes/kr210r3300kultra/link_a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; visual mesh filename=package://kuka_kr210_support/meshes/kr210r3300kultra/link_a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
- added link link_a4, mass 5.113; collision mesh filename=package://kuka_kr210_support/meshes/kr210r3300kultra/link_a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; visual mesh filename=package://kuka_kr210_support/meshes/kr210r3300kultra/link_a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
- added link link_a5, mass 11.495; collision mesh filename=package://kuka_kr210_support/meshes/kr210r3300kultra/link_a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; visual mesh filename=package://kuka_kr210_support/meshes/kr210r3300kultra/link_a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
- added link link_a6, mass 0.64081; collision mesh filename=package://kuka_kr210_support/meshes/kr210r3300kultra/link_a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; visual mesh filename=package://kuka_kr210_support/meshes/kr210r3300kultra/link_a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
- link base_link: geometry collision mesh filename=package://kuka_kr210_support/meshes/kr210r3300kultra/base_l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; visual mesh filename=package://kuka_kr210_support/meshes/kr210r3300kultra/base_l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
Joints:
- removed joint a1
- removed joint a2
- removed joint a3
- removed joint a4
- removed joint a5
- removed joint a6
- added joint joint_a1: type revolute, parent base_link, child link_a1, origin xyz=0 0.01 0.21464 rpy=-6.123E-17 5.6221E-20 0.00091819, axis 0 0 -1, limit lower=-3.2289 upper=3.2289 effort=0 velocity=1.8326
- added joint joint_a2: type revolute, parent link_a1, child link_a2, origin xyz=0.75 -0.01 0.37536 rpy=3.1416 1.5528 -3.1416, axis 0 1 0, limit lower=-2.0944 upper=1.2217 effort=0 velocity=1.7628
- added joint joint_a3: type revolute, parent link_a2, child link_a3, origin xyz=0 0.01 1.35 rpy=3.1416 -1.5469 -3.1416, axis 0 1 0, limit lower=-2.0944 upper=2.7053 effort=0 velocity=1.8675
- added joint joint_a4: type revolute, parent link_a3, child link_a4, origin xyz=0.92112 -0.01 -0.041 rpy=3.9824E-19 -0.15463 -1.5708, axis 0 -1 0, limit lower=-6.1087 upper=6.1087 effort=0 velocity=2.3736
- added joint joint_a5: type revolute, parent link_a4, child link_a5, origin xyz=-0.01 0.27888 0 rpy=-8.0493E-16 0.0059619 1.5708, axis 0 1 0, limit lower=-2.138 upper=2.138 effort=0 velocity=2.2515
- added joint joint_a6: type revolute, parent link_a5, child link_a6, origin xyz=0.205 -6.1532E-05 0.0011076 rpy=0.11099 0 0, axis -1 0 0, limit lower=-6.1087 upper=6.1087 effort=0 velocity=3.5954

Commit message: Update joint rpy to 0.0 or pi/2

File: kuka_kr210_support/urdf/kr210r3300kultra.urdf (robot description, URDF)
Before this commit: robot KR210_R3300_K_ultra, 7 links, 6 joints
Joints:
- joint joint_a1: origin xyz=0 0.01 0.21464 rpy=-6.123E-17 5.6221E-20 0.00091819 -> xyz=0 0.01 0.21464 rpy=0.0 0.0 0.0
- joint joint_a2: origin xyz=0.75 -0.01 0.37536 rpy=3.1416 1.5528 -3.1416 -> xyz=0.75 -0.01 0.37536 rpy=0.0 1.570796 0.0
- joint joint_a3: origin xyz=0 0.01 1.35 rpy=3.1416 -1.5469 -3.1416 -> xyz=0 0.01 1.35 rpy=0.0 -1.570796 0.0
- joint joint_a4: origin xyz=0.92112 -0.01 -0.041 rpy=3.9824E-19 -0.15463 -1.5708 -> xyz=0.92112 -0.01 -0.041 rpy=0.0 0.0 -1.570796
- joint joint_a5: origin xyz=-0.01 0.27888 0 rpy=-8.0493E-16 0.0059619 1.5708 -> xyz=-0.01 0.27888 0 rpy=0.0 0.0 1.570796
- joint joint_a6: origin xyz=0.205 -6.1532E-05 0.0011076 rpy=0.11099 0 0 -> xyz=0.205 0.0 0.0011076 rpy=0.0 0 0

Commit message: Add tool0 link

File: kuka_kr210_support/urdf/kr210r3300kultra.urdf (robot description, URDF)
Before this commit: robot KR210_R3300_K_ultra, 7 links, 6 joints
Links:
- added link tool0
Joints:
- added joint link_a6-tool0: type fixed, parent link_a6, child tool0, origin xyz=0.035 0 0 rpy=0 0 0
